Commit message: UPD: Prop params

File: assets/urdf/cylinder/cylinder.urdf (robot description, URDF)
Before this commit: robot cylinder_v, 1 links, 0 joints
Links:
- link cylinder_v__link_0: mass 1 -> 0.072; geometry collision cylinder length=0.15 radius=0.015; visual cylinder length=0.15 radius=0.015
