Commit message: ADD: Moonrock Prop

File: assets/urdf/donut_1/donut.urdf (robot description, URDF)
Before this commit: robot donut_1, 1 links, 0 joints
Links:
- link donut_1__link_6: mass 0 -> 0.25

File: assets/urdf/sphere/sphere.urdf (robot description, URDF)
Before this commit: robot sphere_v, 1 links, 0 joints
Links:
- link sphere_v__link_1: mass 1 -> 0.25
