Commit message: UPD: Randomly generated rocks

File: assets/rocks/urdf/0.urdf (robot description, URDF)
Before this commit: robot rock, 1 links, 0 joints
Links:
- link rock: geometry collision mesh filename=package://rocks/visual/0.dae scale=1 1 1; visual mesh filename=package://rocks/visual/0.dae scale=1 1 1

File: assets/rocks/urdf/1.urdf (robot description, URDF)
Before this commit: robot rock, 1 links, 0 joints
Links:
- link rock: geometry collision mesh filename=package://rocks/visual/1.dae scale=1 1 1; visual mesh filename=package://rocks/visual/1.dae scale=1 1 1

File: assets/rocks/urdf/10.urdf (robot description, URDF)
Before this commit: robot rock, 1 links, 0 joints
Links:
- link rock: geometry collision mesh filename=package://rocks/visual/10.dae scale=1 1 1; visual mesh filename=package://rocks/visual/10.dae scale=1 1 1

File: assets/rocks/urdf/11.urdf (robot description, URDF)
Before this commit: robot rock, 1 links, 0 joints
Links:
- link rock: geometry collision mesh filename=package://rocks/visual/11.dae scale=1 1 1; visual mesh filename=package://rocks/visual/11.dae scale=1 1 1

File: assets/rocks/urdf/12.urdf (robot description, URDF)
Before this commit: robot rock, 1 links, 0 joints
Links:
- link rock: geometry collision mesh filename=package://rocks/visual/12.dae scale=1 1 1; visual mesh filename=package://rocks/visual/12.dae scale=1 1 1

File: assets/rocks/urdf/13.urdf (robot description, URDF)
Before this commit: robot rock, 1 links, 0 joints
Links:
- link rock: geometry collision mesh filename=package://rocks/visual/13.dae scale=1 1 1; visual mesh filename=package://rocks/visual/13.dae scale=1 1 1

File: assets/rocks/urdf/14.urdf (robot description, URDF)
Before this commit: robot rock, 1 links, 0 joints
Links:
- link rock: geometry collision mesh filename=package://rocks/visual/14.dae scale=1 1 1; visual mesh filename=package://rocks/visual/14.dae scale=1 1 1

File: assets/rocks/urdf/15.urdf (robot description, URDF)
Before this commit: robot rock, 1 links, 0 joints
Links:
- link rock: geometry collision mesh filename=package://rocks/visual/15.dae scale=1 1 1; visual mesh filename=package://rocks/visual/15.dae scale=1 1 1

File: assets/rocks/urdf/16.urdf (robot description, URDF)
Before this commit: robot rock, 1 links, 0 joints
Links:
- link rock: geometry collision mesh filename=package://rocks/visual/16.dae scale=1 1 1; visual mesh filename=package://rocks/visual/16.dae scale=1 1 1

File: assets/rocks/urdf/17.urdf (robot description, URDF)
Before this commit: robot rock, 1 links, 0 joints
Links:
- link rock: geometry collision mesh filename=package://rocks/visual/17.dae scale=1 1 1; visual mesh filename=package://rocks/visual/17.dae scale=1 1 1

File: assets/rocks/urdf/18.urdf (robot description, URDF)
Before this commit: robot rock, 1 links, 0 joints
Links:
- link rock: geometry collision mesh filename=package://rocks/visual/18.dae scale=1 1 1; visual mesh filename=package://rocks/visual/18.dae scale=1 1 1

File: assets/rocks/urdf/19.urdf (robot description, URDF)
Before this commit: robot rock, 1 links, 0 joints
Links:
- link rock: geometry collision mesh filename=package://rocks/visual/19.dae scale=1 1 1; visual mesh filename=package://rocks/visual/19.dae scale=1 1 1

File: assets/rocks/urdf/2.urdf (robot description, URDF)
Before this commit: robot rock, 1 links, 0 joints
Links:
- link rock: geometry collision mesh filename=package://rocks/visual/2.dae scale=1 1 1; visual mesh filename=package://rocks/visual/2.dae scale=1 1 1

File: assets/rocks/urdf/20.urdf (robot description, URDF)
Before this commit: robot rock, 1 links, 0 joints
Links:
- link rock: geometry collision mesh filename=package://rocks/visual/20.dae scale=1 1 1; visual mesh filename=package://rocks/visual/20.dae scale=1 1 1

File: assets/rocks/urdf/21.urdf (robot description, URDF)
Before this commit: robot rock, 1 links, 0 joints
Links:
- link rock: geometry collision mesh filename=package://rocks/visual/21.dae scale=1 1 1; visual mesh filename=package://rocks/visual/21.dae scale=1 1 1

File: assets/rocks/urdf/22.urdf (robot description, URDF)
Before this commit: robot rock, 1 links, 0 joints
Links:
- link rock: geometry collision mesh filename=package://rocks/visual/22.dae scale=1 1 1; visual mesh filename=package://rocks/visual/22.dae scale=1 1 1

File: assets/rocks/urdf/23.urdf (robot description, URDF)
Before this commit: robot rock, 1 links, 0 joints
Links:
- link rock: geometry collision mesh filename=package://rocks/visual/23.dae scale=1 1 1; visual mesh filename=package://rocks/visual/23.dae scale=1 1 1

File: assets/rocks/urdf/24.urdf (robot description, URDF)
Before this commit: robot rock, 1 links, 0 joints
Links:
- link rock: geometry collision mesh filename=package://rocks/visual/24.dae scale=1 1 1; visual mesh filename=package://rocks/visual/24.dae scale=1 1 1

File: assets/rocks/urdf/25.urdf (robot description, URDF)
Before this commit: robot rock, 1 links, 0 joints
Links:
- link rock: geometry collision mesh filename=package://rocks/visual/25.dae scale=1 1 1; visual mesh filename=package://rocks/visual/25.dae scale=1 1 1

File: assets/rocks/urdf/26.urdf (robot description, URDF)
Before this commit: robot rock, 1 links, 0 joints
Links:
- link rock: geometry collision mesh filename=package://rocks/visual/26.dae scale=1 1 1; visual mesh filename=package://rocks/visual/26.dae scale=1 1 1
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
Commit message: ADD: Friction options and New rocks

File: assets/rocks/urdf/0.urdf (robot description, URDF)
Before this commit: robot rock, 1 links, 0 joints
Links:
- link rock: mass 0.25 -> 0.241

File: assets/rocks/urdf/1.urdf (robot description, URDF)
Before this commit: robot rock, 1 links, 0 joints
Links:
- link rock: mass 0.25 -> 0.303

File: assets/rocks/urdf/10.urdf (robot description, URDF)
Before this commit: robot rock, 1 links, 0 joints
Links:
- link rock: mass 0.25 -> 0.214

File: assets/rocks/urdf/11.urdf (robot description, URDF)
Before this commit: robot rock, 1 links, 0 joints
Links:
- link rock: mass 0.25 -> 0.343

File: assets/rocks/urdf/12.urdf (robot description, URDF)
Before this commit: robot rock, 1 links, 0 joints
Links:
- link rock: mass 0.25 -> 0.231

File: assets/rocks/urdf/13.urdf (robot description, URDF)
Before this commit: robot rock, 1 links, 0 joints
Links:
- link rock: mass 0.25 -> 0.288

File: assets/rocks/urdf/14.urdf (robot description, URDF)
Before this commit: robot rock, 1 links, 0 joints
Links:
- link rock: mass 0.25 -> 0.327

File: assets/rocks/urdf/15.urdf (robot description, URDF)
Before this commit: robot rock, 1 links, 0 joints
Links:
- link rock: mass 0.25 -> 0.298

File: assets/rocks/urdf/16.urdf (robot description, URDF)
Before this commit: robot rock, 1 links, 0 joints
Links:
- link rock: mass 0.25 -> 0.308

File: assets/rocks/urdf/17.urdf (robot description, URDF)
Before this commit: robot rock, 1 links, 0 joints
Links:
- link rock: mass 0.25 -> 0.322

File: assets/rocks/urdf/18.urdf (robot description, URDF)
Before this commit: robot rock, 1 links, 0 joints
Links:
- link rock: mass 0.25 -> 0.204

File: assets/rocks/urdf/19.urdf (robot description, URDF)
Before this commit: robot rock, 1 links, 0 joints
Links:
- link rock: mass 0.25 -> 0.267

File: assets/rocks/urdf/2.urdf (robot description, URDF)
Before this commit: robot rock, 1 links, 0 joints
Links:
- link rock: mass 0.25 -> 0.302

File: assets/rocks/urdf/20.urdf (robot description, URDF)
Before this commit: robot rock, 1 links, 0 joints
Links:
- link rock: mass 0.25 -> 0.350

File: assets/rocks/urdf/21.urdf (robot description, URDF)
Before this commit: robot rock, 1 links, 0 joints
Links:
- link rock: mass 0.25 -> 0.226

File: assets/rocks/urdf/22.urdf (robot description, URDF)
Before this commit: robot rock, 1 links, 0 joints
Links:
- link rock: mass 0.25 -> 0.215

File: assets/rocks/urdf/23.urdf (robot description, URDF)
Before this commit: robot rock, 1 links, 0 joints
Links:
- link rock: mass 0.25 -> 0.343

File: assets/rocks/urdf/24.urdf (robot description, URDF)
Before this commit: robot rock, 1 links, 0 joints
Links:
- link rock: mass 0.25 -> 0.298

File: assets/rocks/urdf/25.urdf (robot description, URDF)
Before this commit: robot rock, 1 links, 0 joints
Links:
- link rock: mass 0.25 -> 0.335

File: assets/rocks/urdf/26.urdf (robot description, URDF)
Before this commit: robot rock, 1 links, 0 joints
Links:
- link rock: mass 0.25 -> 0.216
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